File: input_stage_SIG-.sch (KiCad schematic (older format))
At the start: 39 parts, among them Q301 BC856BS, Q302 MMBFJ112, Q303 MMBFJ112, Q304 LS844, Q305 JFE2140DR, Q306 2N7002HSX, Q307 BC846BDW1

Commit message: work continues
Parts:
- Q304: symbol LS844-SOT-23-6L-CT:LS844-SOT-23-6L-CT -> input_buffer_discrete_eval-rescue:LS844-SOT-23-6L-CT-LS844-SOT-23-6L-CT
- Q305: symbol JFE2140DR:JFE2140DR -> input_buffer_discrete_eval-rescue:JFE2140DR-JFE2140DR
- Q306: symbol 2N7002HSX:2N7002HSX -> input_buffer_discrete_eval-rescue:2N7002HSX-2N7002HSX
Changed lines of the file:
@@
 $EndComp
 $Comp
-L LS844-SOT-23-6L-CT:LS844-SOT-23-6L-CT Q?
+L input_buffer_discrete_eval-rescue:LS844-SOT-23-6L-CT-LS844-SOT-23-6L-CT Q?
 U 1 1 64914579
 P 3050 3900
@@
 $EndComp
 $Comp
-L JFE2140DR:JFE2140DR IC?
+L input_buffer_discrete_eval-rescue:JFE2140DR-JFE2140DR IC?
 U 1 1 64652E48
 P 3000 4850
@@
 $EndComp
 $Comp
-L 2N7002HSX:2N7002HSX Q?
+L input_buffer_discrete_eval-rescue:2N7002HSX-2N7002HSX Q?
 U 1 1 646552FE
 P 3050 5900
 AR Path="/64618ED1/646552FE" Ref="Q?"  Part="1"
 AR Path="/647CF58A/646552FE" Ref="Q306"  Part="1"
+AR Path="/646552FE" Ref="Q306"  Part="1"
 F 0 "Q306" H 3500 6165 50  0000 C CNN
 F 1 "2N7002HSX" H 3500 6074 50  0000 C CNN

Commit message: work continues
Parts:
- Q305: footprint (none) -> Package_SO:SOIC-8_3.9x4.9mm_P1.27mm
Changed lines of the file:
@@
 F 0 "Q305" H 3500 5115 50  0000 C CNN
 F 1 "JFE2140DR" H 3500 5024 50  0000 C CNN
-F 2 "" H 3850 4950 50  0001 L CNN
+F 2 "Package_SO:SOIC-8_3.9x4.9mm_P1.27mm" H 3850 4950 50  0001 L CNN
 F 3 "https://www.ti.com/lit/ds/symlink/jfe2140.pdf?ts=1633964558921" H 3850 4850 50  0001 L CNN
 F 4 "JFE2140 Ultra-Low Noise, Matched, Dual, Low-Gate Current, Discrete, Audio, NChannel JFET" H 3850 4750 50  0001 L CNN "Description"
