File: output_stage.sch (KiCad schematic (older format))
At the start: 19 parts, among them J401 OUT, Q401 BC856, Q402 BC846, Q403 BCP53, Q404 BCP56, Q405 BC856, Q406 BC846, Q407 BCP53, Q408 BCP56

Commit message: work continues
Parts:
- J401: footprint (none) -> TerminalBlock_Phoenix:TerminalBlock_Phoenix_PT-1,5-3-3.5-H_1x03_P3.50mm_Horizontal
Changed lines of the file:
@@
 F 0 "J401" H 7918 3675 50  0000 C CNN
 F 1 "OUT" H 7918 3766 50  0000 C CNN
-F 2 "" H 8000 4000 50  0001 C CNN
+F 2 "TerminalBlock_Phoenix:TerminalBlock_Phoenix_PT-1,5-3-3.5-H_1x03_P3.50mm_Horizontal" H 8000 4000 50  0001 C CNN
 F 3 "~" H 8000 4000 50  0001 C CNN
 	1    8000 4000
