File: psu.sch (KiCad schematic (older format))
At the start: 21 parts, among them J501 POWER, U1 LM317_TO-252, U2 LM337_TO252

Commit message: work continues
Parts:
- C503, C504: footprint (none) -> Capacitor_THT:CP_Radial_D6.3mm_P2.50mm
- C505, C506: footprint (none) -> Capacitor_THT:CP_Radial_D10.0mm_P5.00mm
Changed lines of the file:
@@
 F 0 "C503" H 5088 3796 50  0000 L CNN
 F 1 "47uF" H 5088 3705 50  0000 L CNN
-F 2 "" H 5000 3750 50  0001 C CNN
+F 2 "Capacitor_THT:CP_Radial_D6.3mm_P2.50mm" H 5000 3750 50  0001 C CNN
 F 3 "~" H 5000 3750 50  0001 C CNN
 	1    5000 3750
@@
 F 0 "C505" H 5588 3546 50  0000 L CNN
 F 1 "470uF" H 5588 3455 50  0000 L CNN
-F 2 "" H 5500 3500 50  0001 C CNN
+F 2 "Capacitor_THT:CP_Radial_D10.0mm_P5.00mm" H 5500 3500 50  0001 C CNN
 F 3 "~" H 5500 3500 50  0001 C CNN
 	1    5500 3500
@@
 F 0 "C504" H 5088 4296 50  0000 L CNN
 F 1 "47uF" H 5088 4205 50  0000 L CNN
-F 2 "" H 5000 4250 50  0001 C CNN
+F 2 "Capacitor_THT:CP_Radial_D6.3mm_P2.50mm" H 5000 4250 50  0001 C CNN
 F 3 "~" H 5000 4250 50  0001 C CNN
 	1    5000 4250
@@
 F 0 "C506" H 5588 4546 50  0000 L CNN
 F 1 "470uF" H 5588 4455 50  0000 L CNN
-F 2 "" H 5500 4500 50  0001 C CNN
+F 2 "Capacitor_THT:CP_Radial_D10.0mm_P5.00mm" H 5500 4500 50  0001 C CNN
 F 3 "~" H 5500 4500 50  0001 C CNN
 	1    5500 4500

Commit message: work continues
Parts:
- D501, D502, D503, D504: footprint (none) -> Diode_SMD:D_SMA_Handsoldering
- J501: footprint (none) -> TerminalBlock_Phoenix:TerminalBlock_Phoenix_PT-1,5-3-3.5-H_1x03_P3.50mm_Horizontal
Changed lines of the file:
@@
 F 0 "J501" H 2418 4317 50  0000 C CNN
 F 1 "POWER" H 2418 4226 50  0000 C CNN
-F 2 "" H 2500 4000 50  0001 C CNN
+F 2 "TerminalBlock_Phoenix:TerminalBlock_Phoenix_PT-1,5-3-3.5-H_1x03_P3.50mm_Horizontal" H 2500 4000 50  0001 C CNN
 F 3 "~" H 2500 4000 50  0001 C CNN
 	1    2500 4000
@@
 F 0 "D501" H 4000 2817 50  0000 C CNN
 F 1 "M7" H 4000 2726 50  0000 C CNN
-F 2 "" H 4000 2600 50  0001 C CNN
+F 2 "Diode_SMD:D_SMA_Handsoldering" H 4000 2600 50  0001 C CNN
 F 3 "~" H 4000 2600 50  0001 C CNN
 	1    4000 2600
@@
 F 0 "D503" V 4954 3330 50  0000 L CNN
 F 1 "M7" V 5045 3330 50  0000 L CNN
-F 2 "" H 5000 3250 50  0001 C CNN
+F 2 "Diode_SMD:D_SMA_Handsoldering" H 5000 3250 50  0001 C CNN
 F 3 "~" H 5000 3250 50  0001 C CNN
 	1    5000 3250
@@
 F 0 "D504" V 4954 4830 50  0000 L CNN
 F 1 "M7" V 5045 4830 50  0000 L CNN
-F 2 "" H 5000 4750 50  0001 C CNN
+F 2 "Diode_SMD:D_SMA_Handsoldering" H 5000 4750 50  0001 C CNN
 F 3 "~" H 5000 4750 50  0001 C CNN
 	1    5000 4750
@@
 F 0 "D502" H 4000 5383 50  0000 C CNN
 F 1 "M7" H 4000 5474 50  0000 C CNN
-F 2 "" H 4000 5600 50  0001 C CNN
+F 2 "Diode_SMD:D_SMA_Handsoldering" H 4000 5600 50  0001 C CNN
 F 3 "~" H 4000 5600 50  0001 C CNN
 	1    4000 5600
