File: rf_emi_filter.sch (KiCad schematic (older format))
At the start: 22 parts, among them J101 SIG_IN

Commit message: work continues
Parts:
- removed JP103: GND_lift, Jumper:SolderJumper-2_P1.3mm_Open_RoundedPad1.0x1.5mm, symbol Device:Jumper_NO_Small
- removed R103: 2M2, Resistor_SMD:R_0805_2012Metric_Pad1.15x1.40mm_HandSolder, symbol Device:R_Small
- removed R104: 47K, Resistor_SMD:R_0805_2012Metric_Pad1.15x1.40mm_HandSolder, symbol Device:R_Small
- R105: value 47K -> 2M2; footprint Resistor_SMD:R_0805_2012Metric_Pad1.15x1.40mm_HandSolder -> (none)
- renumbered JP104 to JP103, JP105 to JP104, JP106 to JP105, R106 to R103, R107 to R104, R108 to R106, R109 to R107
Connections:
- net GND: now also JP103.2, JP104.1, R105.2
- net at JP105.1, R106.2, R107.1: now also R105.1; no longer JP103.2, JP104.1
- net at C102.2, C104.2, JP102.1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: no longer R105.2
Other:
- moved on the sheet: C103, C104, C105, C106, JP101, JP102, JP103, JP104, R103, R104

Commit message: work continues
Parts:
- J101: footprint (none) -> Connector_Audio:Jack_XLR_Neutrik_NC3FAAH2_Horizontal
Changed lines of the file:
@@
 F 0 "J101" V 2046 4228 50  0000 L CNN
 F 1 "SIG_IN" V 1955 4228 50  0000 L CNN
-F 2 "" H 2000 4000 50  0001 C CNN
+F 2 "Connector_Audio:Jack_XLR_Neutrik_NC3FAAH2_Horizontal" H 2000 4000 50  0001 C CNN
 F 3 " ~" H 2000 4000 50  0001 C CNN
 	1    2000 4000
